File: dcMotor.kicad_sch (KiCad schematic)
At the start: 125 parts, among them J1 USB_C_Receptacle_USB2.0_16P, J2 USB_C_Receptacle_USB2.0_16P, J3 Conn_ST_STDC14, J6 Conn_01x02_Pin, J7 Conn_01x04_Pin, J8 Conn_01x06_Pin, Q1 AO3400A, SW1 SW_Push, SW2 SW_Push, U1 LMR54406DBVR, U10 MCP6561-OT, U11 NUCLEO-L432KC, U12 NUCLEO-F411RE, U2 NCP718ASNADJT1G, U3 NCP718ASNADJT1G, U5 TLV9152IDR, U6 ER_OLEDM0.91_1x-I2C, U7 STM32G431CBTx, U8 LTH-301-05, U9 DRV8231ADDA

Commit message: changed to A2 and added docu
Parts:
- removed U11: NUCLEO-L432KC, local:MODULE_NUCLEO-L432KC, symbol NUCLEO-L432KC:NUCLEO-L432KC
Connections:
- net GND: now also U12.CN10_32 (AGND), U12.CN10_9 (GND_9), U12.CN7_19 (GND_19), U12.CN7_22 (GND_22), U12.CN7_8 (GND_8)
Other:
- note added: "12V -> 3.3V"
- note added: "5V for HALL-Supply and Back-EMF Measurement do NOT load more than ~30mA"
- note added: "Achtung: Für <>12V: C15850 statt C440198 C1, C29, C30, C37 da für 12V ok und günstiger"
- note added: "Back-EMF measurement"
- note added: "Board Power Supply (+12V)"
- note added: "D2 to not leave uC unpowered when only data connector is plugged in"
- note added: "Debug Header"
- note added: "Display (optional)"
- note added: "MATLAB"
- note added: "MB1136: Nucleo64(F411)"
- note added: "Motor Connector TIM2 configured in CubeMX as "combined channels" in Encoder Mode to measure Motor Hall Encoder Signals"
- note added: "Motor-Driver"
- note added: "No CTR given in Datasheet 1.) At IF = 20mA -> Datasheet guaratees > 0.5mA photocurrent -> estimated worst case CTR ~0.5/20 = 2.5% -> worst case IC @ 10mA LED drive = 240µA -> For Rload = 1k -> Vlow,out = 3.3-240µA*1k = 3.1V -> only 0.2V swing 2.) To guarantee saturation in worst case, Rload must limit Ic to 240µA Rload > (3.3-VCE,sat)/240µA = 13kOhm 3.) Estimate Rload for large enough output swin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"
- note added: "Photo Interruptor"
- note added: "Potentiometer for manual speed control"
- note added: "RM0444 Rev 5 40.4.4 internal PU PD cheapo: Tokmas MBRS340T3G (onsemi@mouser:0,5) Tokmas@JLC: 0,05"
- note added: "Schmitt-Trigger"
- note added: "USB 2 FS -> PC (! DATA only !)"
- note added: "USBC Power, OPTIONAL NOT used for first experiments(only If we want to power the Board with 9/12V via USBC-PD later)"
- note added: "VM: 4.5-V to 33-V supply rail f_{PWM}: 0 - 200kHz logic inputs: 100k internal PD IN1 = IN2 = 0 for t>1.5ms : low power mode IN1 = 1 && IN2 = 0 -> Forward IN1 = 1 && IN2 = 1 -> Slow decay IN1 = 0 && IN2 = 0 -> Fast decay Forward with coast (coast = async. fast decay) : IN1: 1 -> 0, IN2: always 0 Forward with break (break = slow decay) : IN2: 0 -> 1, IN1: always 1 For "manual" Back-EMF measurement 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"
- note added: "Virtual GND for Back-EMF Measurement"
- note added: "shift down the 5V to ~3V3 inkl. speed-up cap"
- note added: "µC"
- note removed: "! DATA only !"
- note removed: "! POWER only !"
- note removed: "12V"
- note removed: "Achtung: Für erste Order C15850 statt C440198 C1, C29, C30, C37 da für 12V ok und günstiger"
- note removed: "No CTR given 1.) At IF = 20mA -> Datasheet guaratees > 0.5mA photocurrent -> estimated worst case CTR ~0.5/20 = 2.5% -> worst case IC @ 10mA LED drive = 240µA -> For Rload = 1k -> Vlow,out = 3.3-240µA*1k = 3.1V -> only 0.2V swing 2.) To guarantee saturation in worst case, Rload must limit Ic to 240µA Rload > (3.3-VCE,sat)/240µA = 13kOhm 3.) Estimate Rload for large enough output swing: For a swin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"
- note removed: "RM0444 Rev 5 40.4.4 internal PU PD"
- note removed: "TIM2 configured in CubeMX as "combined channels" in Encoder Mode to measure Motor Hall Encoder Signals"
- note removed: "VM: 4.5-V to 33-V supply rail f_{PWM}: 0 - 200kHz logic inputs: 100k internal PD IN1 = IN2 = 0 for t>1.5ms : low power mode IN1 = 1 && IN2 = 0 -> Forward IN1 = 1 && IN2 = 1 -> Slow decay IN1 = 0 && IN2 = 0 -> Fast decay FW fast : IN1: 1 -> 0, IN2: always 0 FW slow : IN1: always 1, IN2: 0 -> 1"
- note removed: "here to not leave uC unpowered when only data connector is plugged in"
- note removed: "rail splitting opamp: OPA994"
- note removed: "shift down the 5V to ~3V3 with speed-up cap"
- moved on the sheet: C1, C10, C11, C12, C13, C14, C15, C16, C17, C18, C19, C2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
