File: hw/V1.1/dcMotor.kicad_pcb (KiCad board)
At the start: 2 copper layers, 144.9 x 98 mm, 158 parts, among them J1 USB_C_Receptacle_USB2.0_16P, J2 Conn_01x02_Socket, J3 Conn_ST_STDC14, J4 Conn_01x02_Socket, J6 Conn_01x02_Pin, J7 Conn_01x04_Pin, J8 Conn_01x06_Pin, Q1 AO3400A, SW1 SW_Push, SW2 SW_Push, U1 LMR54406DBVR, U10 MCP6561-OT, U11 TLV9152IDR, U12 NUCLEO-F411RE:NUCLEO-F411RE, U13 INA241A4IDR, U2 NCP718ASNADJT1G, U3 NCP718ASNADJT1G, U5 TLV9152IDR, U6 ER_OLEDM0.91_1x-I2C, U7 STM32G431CBTx, U8 LTH-301-05, U9 DRV8251ADDA

Commit message: some fixes in rigol python script
Parts:
- moved R47 5.84 mm to (163.7, 119.8)
- moved R48 5.84 mm to (163.7, 117.6)
- moved R50 5.84 mm to (163.7, 125.9)
- moved R51 5.84 mm to (163.7, 123.9)
- moved R52 5.84 mm to (163.7, 121.9)
Routing:
- net /IMOTOR: track 170.3 -> 174.2 mm
- net /UMOTOR: track 151.4 -> 155.1 mm
- net Net-(U12A-PA0): track 9.42 -> 11.8 mm
- net /MOTOR-_SENSE: track 149.9 -> 152.3 mm
- net /MOTOR+_SENSE: track 157.6 -> 160.0 mm
- net /EN_PHOTO: track 82.3 -> 84.5 mm
- net Net-(U12A-PA1): track 9.56 -> 11.6 mm
- net Net-(U12A-PC1): track 19.7 -> 21.6 mm
- net Net-(U12A-PA4): track 9.77 -> 11.4 mm
- net Net-(U12A-PC0): track 22.7 -> 23.5 mm
